File: hardware/Ohmmeter/Ohmmeter.kicad_pcb (KiCad board)
At the start: 2 copper layers, 147.3 x 101.6 mm, 68 parts, among them J1 Power, Q1 KT361, Q2 KT361, Q3 KT361, Q4 KT361, Q5 KT361, Q6 2N4401, Q7 2N4401, Q8 BC212B, U1 LM741, U2 LM741, U3 L78L05_TO92, U4 LM741, U5 ATmega8A-PU

Commit message: PCB Fixes.
Parts:
- moved C10 2.62 mm to (193.0, 45.6)
Connections:
- DS1 pad 15: (no net) -> Net-(DS1-Pad15)
- DS1 pad 16: (no net) -> Net-(DS1-Pad16)
- DS1 pad 17: Net-(DS1-Pad17) -> (no net)
- DS1 pad 18: Net-(DS1-Pad18) -> (no net)
- R3 pad 2: Net-(DS1-Pad17) -> Net-(DS1-Pad15)
- R4 pad 2: Net-(DS1-Pad18) -> Net-(DS1-Pad16)
- R7 pad 1: Net-(DS1-Pad17) -> Net-(DS1-Pad15)
- R8 pad 1: Net-(DS1-Pad18) -> Net-(DS1-Pad16)
- U5 pad 4: Net-(DS1-Pad17) -> Net-(DS1-Pad15)
- U5 pad 5: Net-(DS1-Pad18) -> Net-(DS1-Pad16)
Routing:
- net Net-(DS1-Pad16): track 0.00 -> 86.4 mm, vias 0 -> 4
- net Net-(DS1-Pad18): track 81.3 -> 0.00 mm, vias 2 -> 0
- net Net-(DS1-Pad15): track 0.00 -> 81.3 mm, vias 0 -> 4
- net Net-(DS1-Pad17): track 76.2 -> 0.00 mm, vias 2 -> 0
- net +VDC: track 378.5 -> 386.1 mm
- net GND: track 411.5 -> 406.4 mm, vias 25 -> 28
- net ADC: track 170.2 -> 167.6 mm, vias 13 -> 12

Commit message: Switch PNP transistors around where possible - I used them all upside-down!
Parts:
- Q8: value BC212B -> MPSA56-AP
- U5: footprint Package_DIP:DIP-28_W7.62mm_Socket -> Package_DIP:DIP-28_W7.62mm
Connections:
- net +3V3 renamed +3.3V
- U1 pad 1: (no net) -> unconnected-(U1-NULL-Pad1)
- U1 pad 5: (no net) -> unconnected-(U1-NULL-Pad5)
- U1 pad 8: (no net) -> unconnected-(U1-NC-Pad8)
- U2 pad 1: (no net) -> unconnected-(U2-NULL-Pad1)
- U2 pad 5: (no net) -> unconnected-(U2-NULL-Pad5)
- U2 pad 8: (no net) -> unconnected-(U2-NC-Pad8)
- U4 pad 1: (no net) -> unconnected-(U4-NULL-Pad1)
- U4 pad 5: (no net) -> unconnected-(U4-NULL-Pad5)
- U4 pad 8: (no net) -> unconnected-(U4-NC-Pad8)
Other:
- net class Default removed
