File: hardware/Ohmmeter/Ohmmeter.kicad_sch (KiCad schematic)
At the start: 62 parts, among them J1 Power, Q1 KT361, Q2 KT361, Q3 KT361, Q4 KT361, Q5 KT361, Q6 2N4401, Q7 2N4401, Q8 BC212B, U1 LM741, U2 LM741, U3 L78L05_TO92, U4 LM741, U5 ATmega8A-PU

Commit message: Switch PNP transistors around where possible - I used them all upside-down!
Parts:
- Q8: value BC212B -> MPSA56-AP; symbol Device:Q_PNP_CBE -> Device:Q_PNP_EBC
Connections:
- net at DS1.15 (NC): now also R3.2, R7.1, U5.4 (PD2)
- net at DS1.16 (NC): now also R4.2, R8.1, U5.5 (PD3)
Other:
- note added: "Floating 3V voltage reference"
- note added: "The PNP transistors below have their emitter and collectors connected in the 'opposite' order to how they should be, and should be flipped if this design is updated. This will require rework of the board, since the physical transistors are in ECB order so can't just be flipped. This revision works well enough even with the transistors 'reversed' that it's okay for now."
Changed lines of the file:
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@@
     (stroke (width 0) (type default))
+  )
+  (text "Floating 3V \nvoltage reference\n" (at 22.86 132.08 0)
+    (effects (font (size 1.27 1.27)) (justify left bottom))
+  )
+  (text "The PNP transistors below have their emitter and collectors connected in the 'opposite' order\nto how they should be, and should be flipped if this design is updated.\n\nThis will require rework of the board, since the physical transistors are in ECB order so can't just be flipped.\n\nThis revision works well enough even with the transistors 'reversed' that it's okay for now."
+    (at 170.18 80.01 0)
+    (effects (font (size 1.27 1.27)) (justify left bottom))
   )
   (global_label "ADC" (shape input) (at 63.5 72.39 0)
@@
     )
   )
-  (symbol (lib_id "Device:Q_PNP_CBE") (at 71.12 176.53 0) (unit 1)
-    (in_bom yes) (on_board yes) (dnp no)
-    (property "Reference" "Q8" (at 75.9714 175.3616 0)
-      (effects (font (size 1.27 1.27)) (justify left))
-    )
-    (property "Value" "BC212B" (at 75.9714 177.673 0)
-      (effects (font (size 1.27 1.27)) (justify left))
-    )
-    (property "Footprint" "Package_TO_SOT_THT:TO-92_Inline_Wide" (at 76.2 173.99 0)
-      (effects (font (size 1.27 1.27)) hide)
-    )
+  (symbol (lib_id "Device:Q_PNP_EBC") (at 71.12 176.53 0) (mirror x) (unit 1)
+    (in_bom yes) (on_board yes) (dnp no) (fields_autoplaced)
+    (property "Reference" "Q8" (at 76.2 175.895 0)
+      (effects (font (size 1.27 1.27)) (justify left))
+    )
+    (property "Value" "MPSA56-AP" (at 76.2 178.435 0)
+      (effects (font (size 1.27 1.27)) (justify left))
+    )
+    (property "Footprint" "Package_TO_SOT_THT:TO-92_Inline_Wide" (at 76.2 179.07 0)
+      (effects (font (size 1.27 1.27)) hide)
+    )

Commit message: Better comments.
Connections:
- net at DS1.15 (NC): now also R3.2, R7.1, U5.4 (PD2)
- net at DS1.16 (NC): now also R4.2, R8.1, U5.5 (PD3)
Other:
- note added: "Floating ~3V power supply"
- note removed: "Floating 3V voltage reference"
Changed lines of the file:
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@@
     (stroke (width 0) (type default))
   )
-  (text "Floating 3V \nvoltage reference\n" (at 22.86 132.08 0)
+  (text "Floating ~3V \npower supply\n" (at 22.86 132.08 0)
     (effects (font (size 1.27 1.27)) (justify left bottom))
   )
